File: BarbaraPCB/BarbaraPCB.kicad_pcb (KiCad board)
At the start: 2 copper layers, 195.3 x 125.5 mm, 139 parts, among them J1 Conn_01x05_Pin, J2 Conn_01x05_Pin, J3 Conn_01x05_Pin_reversed, J4 Conn_01x05_Pin_reversed, SW1 SW_Push, SW10 SW_Push, SW11 SW_Push, SW12 SW_Push, SW13 SW_Push, SW14 SW_Push, SW15 SW_Push, SW16 SW_Push, SW17 SW_Push, SW18 SW_Push, SW19 SW_Push, SW2 SW_Push, SW20 SW_Push, SW21 SW_Push_1.5u, SW22 SW_Push, SW23 SW_Push, SW24 SW_Push, SW25 SW_Push, SW26 SW_Push, SW27 SW_Push, SW28 SW_Push, SW29 SW_Push_1.5u, SW3 SW_Push, SW30 SW_Push, SW31 SW_Push, SW32 SW_Push, SW33 SW_Push, SW34 SW_Push, SW35 SW_Push_1.25u, SW36 SW_Push_1.75u, SW37 SW_Push_1.75u, SW38 SW_Push_1.25u, SW39 SW_Push, SW4 SW_Push, SW40 SW_Push, SW41 SW_Push, SW42 SW_Push, SW43 SW_Push, SW44 SW_Push, SW45 SW_Push_1.5u, SW46 SW_Push_1.5u, SW47 SW_Push_1.5u, SW48 SW_Push_1.5u, SW49 SW_Push, SW5 SW_Push, SW50 SW_Push, SW51 SW_Push, SW52 SW_Push, SW53 SW_Push, SW54 SW_Push_1.25u, SW55 SW_Push_1.75u, SW56 SW_Push_1.75u, SW57 SW_Push_1.25u, SW58 SW_Push, SW59 SW_Push, SW6 SW_Push, SW60 SW_Push, SW61 SW_Push, SW62 SW_Push, SW63 SW_Push, SW64 SW_Push_1.5u, SW65 SW_Push_1.5u, SW66 SW_Push_1.5u, SW67 SW_Push_1.5u, SW7 SW_Push, SW8 SW_Push, SW9 SW_Push, U2 RP2040-Matrix

Commit message: Soundbauteile hinzugefügt
Parts:
- removed U2: RP2040-Matrix, TFL:RP2040-Gemini-BigHole
- added BZ1: Buzzer, Buzzer_Beeper:MagneticBuzzer_StarMicronics_QMB-105, B.Cu at (30.6, 46.4)
- added C1: 100n, Capacitor_THT:C_Disc_D5.0mm_W2.5mm_P5.00mm, F.Cu at (27.1, 0.02)
- added C2: 100n, Capacitor_SMD:C_0805_2012Metric_Pad1.18x1.45mm_HandSolder, F.Cu at (34.4, 3.55)
- added D48: 1N4148, TFL:Diode-dual, F.Cu at (30.7, -8.69)
- added J5: Connector for PAM8403 Amp, Connector_PinHeader_2.54mm:PinHeader_1x04_P2.54mm_Vertical, F.Cu at (23.2, -7.73)
- added Q2: PN2222A, Package_TO_SOT_THT:TO-92_Inline, F.Cu at (27.5, 5.30)
- added R1: 1K, TFL:Diode-dual, F.Cu at (30.7, -6.01)
- added R2: 1K, TFL:Diode-dual, F.Cu at (30.7, -3.34)
- added U1: RP2040-Matrix, TFL:RP2040-Gemini-BigHole, F.Cu at (57.2, 36.8)
- moved D1 1.30 mm to (46.3, 38.1)
- moved D6 1.26 mm to (142.9, 38.1)
- moved D5 1.25 mm to (123.8, 38.1)
- moved D2 1.16 mm to (67.8, 38.1)
Other:
- outline, holes or cut-outs redrawn

Commit message: Silk und diverse Kleinigkeiten. Productionready?!
Parts:
- added REF**: Clacktales_9mm_whiteSilk, Silkscreen:Clacktales_9mm_whiteSilk, B.Cu at (169.2, 47.8)
- added Ref**: Val**, Silkscreen:BarBara Kopf only 3,5u, F.Cu at (130.2, 64.1)
- added Ref**: Val**, Silkscreen:BarBara minimal Barbar, B.Cu at (123.9, 140.8)
- added Ref**: Val**, Silkscreen:Moinboards new logo 10mm, B.Cu at (157.8, 48.3)
- added Ref**: Val**, Silkscreen:BarBara minimal only big, B.Cu at (125.6, 65.5)
- added Ref**: Val**, Silkscreen:BarBara Kopf only 1u, B.Cu at (263.3, 66.1)
- 1k: renamed from R2; footprint TFL:Diode-dual -> TFL:Resistor-dual; moved to B.Cu
- 1k: renamed from R1; footprint TFL:Diode-dual -> TFL:Resistor-dual; moved to B.Cu
- C1, C2, D48, J5, U1: moved to B.Cu
- PN2222A: renamed from Q2; moved to B.Cu
- moved J5 87.9 mm to (28.6, 80.0)
- moved 1k 70.7 mm to (40.5, 66.7)
- moved C1 66.9 mm to (33.3, 66.7), turned to 180 degrees
- moved D48 65.9 mm to (28.6, 57.1), turned to 90 degrees
- moved C2 63.2 mm to (31.0, 66.7), turned to 180 degrees
- moved 1k 59.6 mm to (47.6, 51.1)
- moved PN2222A 45.5 mm to (44.1, 47.6), turned to 180 degrees
- moved D36 5.01 mm to (161.9, 97.6)
- moved D34 4.32 mm to (123.8, 99.4)
- moved D32 3.92 mm to (70.3, 97.6)
- moved D31 3.81 mm to (50.0, 97.6)
- moved D35 3.26 mm to (147.6, 99.5)
- moved D33 3.10 mm to (100.0, 100.5)
- moved D37 2.52 mm to (176.2, 97.6)
- turned U1 to 180 degrees
Connections:
- 1k pad 1: Net-(U1-P13) -> Net-(U1-P9)
- 1k pad 1: Net-(U1-P14) -> Net-(U1-P8)
- U1 pad 13: unconnected-(U1-P3-Pad13) -> row0
- U1 pad 14: unconnected-(U1-P4-Pad14) -> col4
- U1 pad 15: unconnected-(U1-P5-Pad15) -> col3
- U1 pad 16: unconnected-(U1-P6-Pad16) -> col2
- U1 pad 17: unconnected-(U1-P7-Pad17) -> col1
- U1 pad 18: unconnected-(U1-P8-Pad18) -> Net-(U1-P8)
- U1 pad 19: Net-(U1-P13) -> row2
- U1 pad 20: unconnected-(U1-P12-Pad20) -> row3
- U1 pad 21: unconnected-(U1-P11-Pad21) -> col0
- U1 pad 22: unconnected-(U1-P10-Pad22) -> row1
- U1 pad 23: unconnected-(U1-P9-Pad23) -> Net-(U1-P9)
- U1 pad 4: row0 -> row9
- U1 pad 5: unconnected-(U1-P28-Pad5) -> row8
- U1 pad 6: unconnected-(U1-P27-Pad6) -> row7
- U1 pad 7: unconnected-(U1-P26-Pad7) -> row6
- U1 pad 8: unconnected-(U1-P15-Pad8) -> row5
- U1 pad 9: Net-(U1-P14) -> row4
Routing:
- net row8: track 0.00 -> 257.6 mm
- net col3: track 0.00 -> 250.3 mm, vias 0 -> 1
- net row9: track 0.00 -> 248.2 mm, vias 0 -> 1
- net row5: track 0.00 -> 246.6 mm, vias 0 -> 1
- net row6: track 0.00 -> 228.8 mm, vias 0 -> 2
- net row4: track 0.00 -> 227.7 mm, vias 0 -> 1
- net col2: track 0.00 -> 207.7 mm
- net Net-(D39-K): track 0.00 -> 204.9 mm
- net row3: track 0.00 -> 192.1 mm, vias 0 -> 4
- net col1: track 0.00 -> 188.4 mm
- net col0: track 0.00 -> 184.7 mm
- net row7: track 0.00 -> 155.3 mm
- net row2: track 0.00 -> 153.8 mm
- net Net-(J4-Pin_5): track 0.00 -> 105.5 mm
- net row1: track 0.00 -> 105.4 mm
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- added copper zone on B.Cu, net GND
- added copper zone on F.Cu, net GND
Other:
- outline, holes or cut-outs redrawn
- board text added: "100n"
- board text added: "5V"
- board text added: "B"
- board text added: "BarBarA by Technofrikus and ggggggg - https://github.com/Technofrikus/BarBarA"
- board text added: "C"
- board text added: "Connector for PAM8403 Amp"
- board text added: "For Gemini Use 3mm header"
- board text added: "GND"
- board text added: "GND (E)"
- board text added: "GND(Sig)"
- board text added: "Reversed!"
- board text added: "Signal (P9)"
